File: kicad/chocV/chocV.kicad_pcb (KiCad board)
At the start: 2 copper layers, 212.5 x 78.7 mm, 84 parts, among them SW1 SW_Push, SW10 SW_Push, SW11 SW_Push, SW12 SW_Push, SW13 SW_Push, SW14 SW_Push, SW15 SW_Push, SW16 SW_Push, SW17 SW_Push, SW18 SW_Push, SW19 SW_Push, SW2 SW_Push, SW20 SW_Push, SW21 SW_Push, SW22 SW_Push, SW23 SW_Push, SW24 SW_Push, SW25 SW_Push, SW26 SW_Push, SW27 SW_Push, SW28 SW_Push, SW29 SW_Push, SW3 SW_Push, SW30 SW_Push, SW31 SW_Push, SW32 SW_Push, SW33 SW_Push, SW34 SW_Push, SW35 SW_Push, SW36 SW_Push, SW37 Reset Switch, SW4 SW_Push, SW5 SW_Push, SW6 SW_Push, SW7 SW_Push, SW8 SW_Push, SW9 SW_Push, U1 Pro-Micro

Commit message: Update PCB, top plate and bottom plate
Add Tactil switch TL3342
Add Slide switch MSK-12C02
Parts:
- removed LOGO1, LOGO2: LOGO, rsu_graphics:bblabs_logo_sml
- added BT1: Device_Battery_Cell, other:PinHeader_1x02_P1.27mm_Vertical, F.Cu at (110.0, 84.6)
- added SW38: Switch_SW_DIP_x01, other:switch_MSK-12C02_smd, B.Cu at (115.1, 94.5)
- SW37: footprint Horizon:SW_Push_6mm -> other:SW_SPST_TL3342; moved to B.Cu
- moved SW37 6.45 mm to (104.9, 92.0), turned to 187 degrees
Connections:
- net GND renamed ground
- U1 pad 24: Net-(U1-Pad24) -> raw
Routing:
- net raw: track 0.00 -> 48.0 mm, vias 0 -> 1
- net reset: track 39.5 -> 54.7 mm, vias 0 -> 1
- net Net-(BT1-Pad1): track 0.00 -> 12.4 mm
- net ground: track 0.00 -> 10.9 mm
